File: pcb/pheromone.sch (KiCad schematic (older format))
At the start: 152 parts, among them J1 USB_C_Receptacle, K1 KEYSW, K10 KEYSW, K11 KEYSW, K12 KEYSW, K13 KEYSW, K14 KEYSW, K15 KEYSW, K16 KEYSW, K17 KEYSW, K18 KEYSW, K19 KEYSW, K2 KEYSW, K20 KEYSW, K21 KEYSW, K22 KEYSW, K23 KEYSW, K24 KEYSW, K25 KEYSW, K26 KEYSW, K27 KEYSW, K28 KEYSW, K29 KEYSW, K3 KEYSW, K30 KEYSW, K31 KEYSW, K32 KEYSW, K33 KEYSW, K34 KEYSW, K35 KEYSW, K36 KEYSW, K37 KEYSW, K38 KEYSW, K39 KEYSW, K4 KEYSW, K40 KEYSW, K41 KEYSW, K42 KEYSW, K43 KEYSW, K44 KEYSW, K45 KEYSW, K46 KEYSW, K47 KEYSW, K48 KEYSW, K49 KEYSW, K5 KEYSW, K50 KEYSW, K51 KEYSW, K52 KEYSW, K53 KEYSW, K54 KEYSW, K55 KEYSW, K56 KEYSW, K57 KEYSW, K58 KEYSW, K59 KEYSW, K6 KEYSW, K60 KEYSW, K61 KEYSW, K62 KEYSW, K63 KEYSW, K7 KEYSW, K8 KEYSW, K9 KEYSW, P1 AVR-ISP-6, SW1 SW_PUSH, U1 ATMEGA32U4, Y1 Crystal_GND24

Commit message: update silks and other stuff
Other:
- moved on the sheet: D64, D65
Changed lines of the file:
@@
 $EndComp
-Wire Wire Line
-	13950 1500 13950 3800
 Wire Wire Line
 	13300 1200 13050 1200
@@
 L Device:D_Zener D64
 U 1 1 5FA8E564
-P 14000 2150
-F 0 "D64" V 13954 2230 50  0000 L CNN
-F 1 "3.6V" V 14045 2230 50  0000 L CNN
-F 2 "Diode_SMD:D_SOD-123" H 14000 2150 50  0001 C CNN
-F 3 "~" H 14000 2150 50  0001 C CNN
-	1    14000 2150
-	0    1    1    0
-$EndComp
-Wire Wire Line
-	14350 2000 14350 1900
+P 14000 2300
+F 0 "D64" V 13954 2380 50  0000 L CNN
+F 1 "3.6V" V 14045 2380 50  0000 L CNN
+F 2 "Diode_SMD:D_SOD-123" H 14000 2300 50  0001 C CNN
+F 3 "~" H 14000 2300 50  0001 C CNN
+	1    14000 2300
+	0    1    1    0
+$EndComp
 $Comp
 L power:GND #PWR0101
 U 1 1 5FC642EA
-P 14200 2300
-F 0 "#PWR0101" H 14200 2050 50  0001 C CNN
-F 1 "GND" H 14205 2127 50  0000 C CNN
-F 2 "" H 14200 2300 50  0001 C CNN
-F 3 "" H 14200 2300 50  0001 C CNN
-	1    14200 2300
+P 14200 2450
+F 0 "#PWR0101" H 14200 2200 50  0001 C CNN
+F 1 "GND" H 14205 2277 50  0000 C CNN
+F 2 "" H 14200 2450 50  0001 C CNN
+F 3 "" H 14200 2450 50  0001 C CNN
+	1    14200 2450
 	1    0    0    -1
 $EndComp
@@
 L Device:D_Zener D65
 U 1 1 5FAD0C3A
-P 14350 2150
-F 0 "D65" V 14304 2230 50  0000 L CNN
-F 1 "3.6v" V 14395 2230 50  0000 L CNN
-F 2 "Diode_SMD:D_SOD-123" H 14350 2150 50  0001 C CNN
-F 3 "~" H 14350 2150 50  0001 C CNN
-	1    14350 2150
+P 14350 2300
+F 0 "D65" V 14304 2380 50  0000 L CNN
+F 1 "3.6v" V 14395 2380 50  0000 L CNN
+F 2 "Diode_SMD:D_SOD-123" H 14350 2300 50  0001 C CNN
+F 3 "~" H 14350 2300 50  0001 C CNN
+	1    14350 2300
 	0    1    1    0
 $EndComp
 Wire Wire Line
 	13050 1900 13200 1900
-Connection ~ 14200 2300
-Wire Wire Line
-	14200 2300 14350 2300
-Wire Wire Line
-	14000 2300 14200 2300
+Connection ~ 14200 2450
+Wire Wire Line
+	14200 2450 14350 2450
+Wire Wire Line
+	14000 2450 14200 2450
 $Comp
 L Connector:USB_C_Receptacle J1
@@
 Wire Wire Line
 	13250 1800 14000 1800
-Wire Wire Line
-	14000 2000 14000 1800
 Connection ~ 13100 1800
 Wire Wire Line
@@
 Text GLabel 14800 1800 2    50   Output ~ 0
 D-
+Wire Wire Line
+	13950 1500 13950 3800
+Wire Wire Line
+	14000 1800 14000 2150
+Wire Wire Line
+	14350 1900 14350 2150
 $EndSCHEMATC
